Commit message: TF tree fixed, no robot in rviz

File: src/xarm_ros2/xarm_description/urdf/camera/gemini2_camera.xacro (robot description, xacro)
@@ -5,5 +5,5 @@
     <!-- define property -->
     <xacro:property name="M_PI" value="3.1415926535897931" />
-    <link name="${prefix}link_eef">
+    <!--<link name="${prefix}link_eef">
       <xacro:common_link_visual
         mesh_filename="camera/gemini2/gemini2"
@@ -15,5 +15,5 @@
         origin_xyz="0 0 0"
         origin_rpy="0 0 0" />
-    </link>
+    </link> -->
     <xacro:if value="${add_gemini2_links}">
       <link name="${prefix}camera_link"></link>

File: src/xarm_ros2/xarm_description/urdf/dual_xarm_device.urdf.xacro (robot description, xacro)
@@ -66,5 +66,5 @@
   <!-- load xarm device -->
   <xacro:include filename="$(find xarm_description)/urdf/xarm_device_macro.xacro" />
-  <!-- <xacro:include filename="$(find xarm_description)/urdf/camera/gemini2_camera.xacro" /> -->
+  <xacro:include filename="$(find xarm_description)/urdf/camera/gemini2_camera.xacro" />
   <xacro:xarm_device prefix="$(arg prefix_1)" hw_ns="$(arg hw_ns)" limited="$(arg limited)"
     effort_control="$(arg effort_control)" velocity_control="$(arg velocity_control)"
@@ -86,5 +86,5 @@
     baud_checkset="$(arg baud_checkset_1)" default_gripper_baud="$(arg default_gripper_baud_1)"
     model1300="$(arg model1300_1)" robot_sn="$(arg robot_sn_1)" mesh_suffix="$(arg mesh_suffix)" kinematics_suffix="$(arg kinematics_suffix_1)" gripper_version="$(arg gripper_version_1)" />
-  <!-- <xacro:gemini2_urdf prefix="$(arg prefix_1)" add_gemini2_links="true"/> -->
+  <xacro:gemini2_urdf prefix="$(arg prefix_1)" add_gemini2_links="true"/>
   <xacro:xarm_device prefix="$(arg prefix_2)" hw_ns="$(arg hw_ns)" limited="$(arg limited)"
     effort_control="$(arg effort_control)" velocity_control="$(arg velocity_control)"
@@ -106,4 +106,4 @@
     baud_checkset="$(arg baud_checkset_2)" default_gripper_baud="$(arg default_gripper_baud_2)"
     model1300="$(arg model1300_2)" robot_sn="$(arg robot_sn_2)" mesh_suffix="$(arg mesh_suffix)" kinematics_suffix="$(arg kinematics_suffix_2)" gripper_version="$(arg gripper_version_2)" />
-  <!-- <xacro:gemini2_urdf prefix="$(arg prefix_2)" add_gemini2_links="true"/> -->
+  <xacro:gemini2_urdf prefix="$(arg prefix_2)" add_gemini2_links="true"/>
 </robot>
