Commit message: URDF cameras are now in Rviz with only issues being L.Camera not connecting via serial number

File: src/xarm_ros2/orbbec_description/urdf/femto_bolt.urdf.xacro (robot description, xacro)
@@ -1,110 +1,109 @@
 <?xml version="1.0"?>
 <robot name="femto_bolt" xmlns:xacro="http://wiki.ros.org/xacro">
-  <!--
-  This is the URDF model for the Orbbec Femto Bolt camera
-  -->
-  <!-- Include files -->
-  <!-- Properties -->
-  <xacro:property name="M_PI" value="3.1415926535897931" />
-  <!-- Dimensions from the provided specifications -->
-  <xacro:property name="cam_width" value="0.1153"/>
-  <xacro:property name="cam_height" value="0.06495"/>
-  <xacro:property name="cam_depth" value="0.04026"/>
-  <xacro:property name="mesh_path" value="package://orbbec_description/meshes/femto_bolt/" />
-  <!-- The following values are approximate but the camera node
-     publishes TF values with actual calibrated camera extrinsic values -->
-  <xacro:property name="base_link_to_link_x" value="0.03645"/>
-  <xacro:property name="base_link_to_link_y" value="0.00198"/>
-  <xacro:property name="base_link_to_link_z" value="0.021"/>
-  <xacro:property name="depth_to_ir_offset" value="0.0"/>
-  <xacro:property name="camera_link_to_depth_rotation_roll" value="-0.0063718"/>
-  <xacro:property name="camera_link_to_depth_rotation_pitch" value="0.1061316"/>
-  <xacro:property name="camera_link_to_depth_rotation_yaw" value="0.000231"/>
-  <xacro:property name="depth_to_color_offset_x" value="-0.0021445322036743163"/>
-  <xacro:property name="depth_to_color_offset_y" value="-0.03267627716064453"/>
-  <xacro:property name="depth_to_color_offset_z" value="-0.0010942233800888062"/>
-  <xacro:property name="depth_to_color_rotation_roll" value="0.006371800289866152"/>
-  <xacro:property name="depth_to_color_rotation_pitch" value="-0.10613163835054795"/>
-  <xacro:property name="depth_to_color_rotation_yaw" value="-0.00023102465978322808"/>
   <xacro:macro name="femto_bolt" params="prefix parent *origin use_nominal_extrinsics:=true">
-    <!-- camera with origin at bottom screw mount -->
-    <joint name="${prefix}_base_joint" type="fixed">
-      <xacro:insert_block name="origin" />
-      <parent link="${parent}"/>
-      <child link="${prefix}_base_link" />
-    </joint>
-    <link name="${prefix}_base_link" >
-      <visual>
-        <origin xyz="0 0 0" rpy="0 0 0"/>
-        <geometry>
-          <mesh filename="${mesh_path}femto_bolt.stl" />
-        </geometry>
-        <material name="">
-          <color rgba="0.792156862745098 0.819607843137255 0.933333333333333 1" />
-        </material>
-      </visual>
-      <collision>
-        <origin xyz="0 0 0" rpy="0 0 0"/>
-        <geometry>
-          <mesh filename="${mesh_path}femto_bolt.stl" />
-        </geometry>
-      </collision>
-      <inertial>
-      <!-- The following are not reliable values, and should not be used for modeling -->
-        <mass value="0.2"/>
-        <origin xyz="0 0 0" rpy="0 0 0"/>
-        <inertia ixx="0.0001" ixy="0.0" ixz="0.0" iyy="0.0001" iyz="0.0" izz="0.0001"/>
-      </inertial>
-    </link>
-    <!-- Camera Link -->
-    <joint name="${prefix}_link_joint" type="fixed">
-      <origin xyz="${base_link_to_link_x} ${base_link_to_link_y} ${base_link_to_link_z}" rpy="0 0 0"/>
-      <parent link="${prefix}_base_link"/>
-      <child link="${prefix}_link"/>
-    </joint>
-    <link name="${prefix}_link" />
-    <!-- Use the nominal extrinsics between camera frames if the calibrated extrinsics aren't being published. e.g. running the device in simulation  -->
-    <xacro:if value="${use_nominal_extrinsics}">
-      <!-- Depth Camera Frame -->
-      <joint name="${prefix}_depth_joint" type="fixed">
-        <origin xyz="0 0 0" rpy="${camera_link_to_depth_rotation_roll} ${camera_link_to_depth_rotation_pitch} ${camera_link_to_depth_rotation_yaw}"/>
-        <parent link="${prefix}_link"/>
-        <child link="${prefix}_depth_frame" />
+    <!--
+    This is the URDF model for the Orbbec Femto Bolt camera
+    -->
+    <!-- Include files -->
+    <!-- Properties -->
+    <xacro:property name="M_PI" value="3.1415926535897931" />
+    <!-- Dimensions from the provided specifications -->
+    <xacro:property name="cam_width" value="0.1153"/>
+    <xacro:property name="cam_height" value="0.06495"/>
+    <xacro:property name="cam_depth" value="0.04026"/>
+    <!-- The following values are approximate but the camera node
+      publishes TF values with actual calibrated camera extrinsic values -->
+    <xacro:property name="base_link_to_link_x" value="0.03645"/>
+    <xacro:property name="base_link_to_link_y" value="0.00198"/>
+    <xacro:property name="base_link_to_link_z" value="0.021"/>
+    <xacro:property name="depth_to_ir_offset" value="0.0"/>
+    <xacro:property name="camera_link_to_depth_rotation_roll" value="-0.0063718"/>
+    <xacro:property name="camera_link_to_depth_rotation_pitch" value="0.1061316"/>
+    <xacro:property name="camera_link_to_depth_rotation_yaw" value="0.000231"/>
+    <xacro:property name="depth_to_color_offset_x" value="-0.0021445322036743163"/>
+    <xacro:property name="depth_to_color_offset_y" value="-0.03267627716064453"/>
+    <xacro:property name="depth_to_color_offset_z" value="-0.0010942233800888062"/>
+    <xacro:property name="depth_to_color_rotation_roll" value="0.006371800289866152"/>
+    <xacro:property name="depth_to_color_rotation_pitch" value="-0.10613163835054795"/>
+    <xacro:property name="depth_to_color_rotation_yaw" value="-0.00023102465978322808"/>
+      <!-- camera with origin at bottom screw mount -->
+      <joint name="${prefix}_base_joint" type="fixed">
+        <xacro:insert_block name="origin" />
+        <parent link="${parent}"/>
+        <child link="${prefix}_base_link" />
       </joint>
-      <link name="${prefix}_depth_frame"/>
-      <joint name="${prefix}_depth_optical_joint" type="fixed">
-        <origin xyz="0 0 0" rpy="${-M_PI/2} 0 ${-M_PI/2}" />
-        <parent link="${prefix}_depth_frame" />
-        <child link="${prefix}_depth_optical_frame" />
+      <link name="${prefix}_base_link" >
+        <visual>
+          <origin xyz="0 0 0" rpy="0 0 0"/>
+          <geometry>
+            <mesh filename="file:///home/cadennurse/xarm_ws/src/xarm_ros2/orbbec_description/meshes/femto_bolt/femto_bolt.stl" />
+          </geometry>
+          <material name="">
+            <color rgba="0.792156862745098 0.819607843137255 0.933333333333333 1" />
+          </material>
+        </visual>
+        <collision>
+          <origin xyz="0 0 0" rpy="0 0 0"/>
+          <geometry>
+            <mesh filename="file:///home/cadennurse/xarm_ws/src/xarm_ros2/orbbec_description/meshes/femto_bolt/femto_bolt.stl" />
+          </geometry>
+        </collision>
+        <inertial>
+        <!-- The following are not reliable values, and should not be used for modeling -->
+          <mass value="0.2"/>
+          <origin xyz="0 0 0" rpy="0 0 0"/>
+          <inertia ixx="0.0001" ixy="0.0" ixz="0.0" iyy="0.0001" iyz="0.0" izz="0.0001"/>
+        </inertial>
+      </link>
+      <!-- Camera Link -->
+      <joint name="${prefix}_link_joint" type="fixed">
+        <origin xyz="${base_link_to_link_x} ${base_link_to_link_y} ${base_link_to_link_z}" rpy="0 0 0"/>
+        <parent link="${prefix}_base_link"/>
+        <child link="${prefix}_link"/>
       </joint>
-      <link name="${prefix}_depth_optical_frame"/>
-      <!-- IR Camera Frame -->
-      <joint name="${prefix}_ir_joint" type="fixed">
-        <origin xyz="0 ${depth_to_ir_offset} 0" rpy="0 0 0" />
-        <parent link="${prefix}_depth_frame" />
-        <child link="${prefix}_ir_frame" />
-      </joint>
-      <link name="${prefix}_ir_frame"/>
-      <joint name="${prefix}_ir_optical_joint" type="fixed">
-        <origin xyz="0 0 0" rpy="${-M_PI/2} 0 ${-M_PI/2}" />
-        <parent link="${prefix}_ir_frame"/>
-        <child link="${prefix}_ir_optical_frame"/>
-      </joint>
-      <link name="${prefix}_ir_optical_frame"/>
-      <!-- Color Camera Frame -->
-      <joint name="${prefix}_color_joint" type="fixed">
-        <origin xyz="${depth_to_color_offset_x} ${depth_to_color_offset_y} ${depth_to_color_offset_z}"
-          rpy="${depth_to_color_rotation_roll} ${depth_to_color_rotation_pitch} ${depth_to_color_rotation_yaw}" />
-        <parent link="${prefix}_depth_frame"/>
-        <child link="${prefix}_color_frame"/>
-      </joint>
-      <link name="${prefix}_color_frame"/>
-      <joint name="${prefix}_color_optical_joint" type="fixed">
-        <origin xyz="0 0 0" rpy="${-M_PI/2} 0 ${-M_PI/2}" />
-        <parent link="${prefix}_color_frame"/>
-        <child link="${prefix}_color_optical_frame"/>
-      </joint>
-      <link name="${prefix}_color_optical_frame"/>
-    </xacro:if>
+      <link name="${prefix}_link" />
+      <!-- Use the nominal extrinsics between camera frames if the calibrated extrinsics aren't being published. e.g. running the device in simulation  -->
+      <xacro:if value="${use_nominal_extrinsics}">
+        <!-- Depth Camera Frame -->
+        <joint name="${prefix}_depth_joint" type="fixed">
+          <origin xyz="0 0 0" rpy="${camera_link_to_depth_rotation_roll} ${camera_link_to_depth_rotation_pitch} ${camera_link_to_depth_rotation_yaw}"/>
+          <parent link="${prefix}_link"/>
+          <child link="${prefix}_depth_frame" />
+        </joint>
+        <link name="${prefix}_depth_frame"/>
+        <joint name="${prefix}_depth_optical_joint" type="fixed">
+          <origin xyz="0 0 0" rpy="${-M_PI/2} 0 ${-M_PI/2}" />
+          <parent link="${prefix}_depth_frame" />
+          <child link="${prefix}_depth_optical_frame" />
+        </joint>
+        <link name="${prefix}_depth_optical_frame"/>
+        <!-- IR Camera Frame -->
+        <joint name="${prefix}_ir_joint" type="fixed">
+          <origin xyz="0 ${depth_to_ir_offset} 0" rpy="0 0 0" />
+          <parent link="${prefix}_depth_frame" />
+          <child link="${prefix}_ir_frame" />
+        </joint>
+        <link name="${prefix}_ir_frame"/>
+        <joint name="${prefix}_ir_optical_joint" type="fixed">
+          <origin xyz="0 0 0" rpy="${-M_PI/2} 0 ${-M_PI/2}" />
+          <parent link="${prefix}_ir_frame"/>
+          <child link="${prefix}_ir_optical_frame"/>
+        </joint>
+        <link name="${prefix}_ir_optical_frame"/>
+        <!-- Color Camera Frame -->
+        <joint name="${prefix}_color_joint" type="fixed">
+          <origin xyz="${depth_to_color_offset_x} ${depth_to_color_offset_y} ${depth_to_color_offset_z}"
+            rpy="${depth_to_color_rotation_roll} ${depth_to_color_rotation_pitch} ${depth_to_color_rotation_yaw}" />
+          <parent link="${prefix}_depth_frame"/>
+          <child link="${prefix}_color_frame"/>
+        </joint>
+        <link name="${prefix}_color_frame"/>
+        <joint name="${prefix}_color_optical_joint" type="fixed">
+          <origin xyz="0 0 0" rpy="${-M_PI/2} 0 ${-M_PI/2}" />
+          <parent link="${prefix}_color_frame"/>
+          <child link="${prefix}_color_optical_frame"/>
+        </joint>
+        <link name="${prefix}_color_optical_frame"/>
+      </xacro:if>
   </xacro:macro>
 </robot>

File: src/xarm_ros2/orbbec_description/urdf/gemini_2.urdf.xacro (robot description, xacro)
@@ -5,5 +5,5 @@
 <robot xmlns:xacro="http://ros.org/wiki/xacro" name="gemini_2">
   <xacro:macro name="gemini_2" params="prefix parent">
-    <xacro:property name="mesh_path" value="package://orbbec_description/meshes/gemini2/" />
+    <xacro:property name="mesh_path" value="file:///home/cadennurse/xarm_ws/src/xarm_ros2/orbbec_description/meshes/gemini2/" />
     <joint name="${prefix}camera_mount_joint" type="fixed">
       <origin xyz="0.06746 -0.0175 0.0237" rpy="3.1415926535897931 -1.5707963267948966 0" />

File: src/xarm_ros2/xarm_description/urdf/dual_xarm_device.urdf.xacro (robot description, xacro)
@@ -109,5 +109,5 @@
   <xacro:gemini_2 prefix="$(arg prefix_2)" parent="$(arg prefix_2)link_eef"/>
    <xacro:femto_bolt prefix="G" parent="world">
-    <origin xyz="0.526 0.290 0.905" rpy="0.0 -1.3090 1.5708"/>
+    <origin xyz="0.526 0.290 0.905" rpy="0.0 -1.3090 0.0"/>
   </xacro:femto_bolt>
 </robot>

Commit message: all three cameras but femto pointcloud work now

File: src/xarm_ros2/orbbec_description/urdf/femto_bolt.urdf.xacro (robot description, xacro)
@@ -78,5 +78,5 @@
         </joint>
         <link name="${prefix}_depth_optical_frame"/>
-        <!-- IR Camera Frame -->
+        <!-- IR Camera Frame
         <joint name="${prefix}_ir_joint" type="fixed">
           <origin xyz="0 ${depth_to_ir_offset} 0" rpy="0 0 0" />
@@ -90,5 +90,5 @@
           <child link="${prefix}_ir_optical_frame"/>
         </joint>
-        <link name="${prefix}_ir_optical_frame"/>
+        <link name="${prefix}_ir_optical_frame"/> -->
         <!-- Color Camera Frame -->
         <joint name="${prefix}_color_joint" type="fixed">

File: src/xarm_ros2/orbbec_description/urdf/gemini_2.urdf.xacro (robot description, xacro)
@@ -88,4 +88,5 @@
       <axis xyz="0 0 0" />
     </joint>
+    <!--
     <link name="${prefix}camera_right_ir_frame">
       <inertial>
@@ -113,5 +114,5 @@
         </material>
       </visual>
-      <!-- <collision>
+       <collision>
         <origin
           xyz="0 0 0"
@@ -120,6 +121,7 @@
           <mesh filename="${mesh_path}camera_infra1_frame.STL" />
         </geometry>
-      </collision> -->
-    </link>
+      </collision>
+    </link> -->
+    <!-- IR Camera Frame
     <joint name="${prefix}camera_right_ir_joint" type="fixed">
       <origin
@@ -154,5 +156,5 @@
           <color rgba="0.792156862745098 0.819607843137255 0.933333333333333 1" />
         </material>
-      </visual>
+      </visual> -->
       <!-- <collision>
         <origin
@@ -162,5 +164,5 @@
           <mesh filename="${mesh_path}camera_infra1_optical_frame.STL" />
         </geometry>
-      </collision> -->
+      </collision>
     </link>
     <joint name="${prefix}camera_right_ir_optical_joint" type="fixed">
@@ -171,5 +173,5 @@
       <child link="${prefix}camera_right_ir_optical_frame" />
       <axis xyz="0 0 0" />
-    </joint>
+    </joint> -->
     <link name="${prefix}camera_color_frame">
       <inertial>
@@ -256,4 +258,5 @@
       <axis xyz="0 0 0" />
     </joint>
+    <!-- LEFT IR camera
     <link name="${prefix}camera_left_ir_frame">
       <inertial>
@@ -280,5 +283,5 @@
           <color rgba="0.792156862745098 0.819607843137255 0.933333333333333 1" />
         </material>
-      </visual>
+      </visual> -->
       <!-- <collision>
         <origin
@@ -288,6 +291,7 @@
           <mesh filename="${mesh_path}camera_infra2_frame.STL" />
         </geometry>
-      </collision> -->
-    </link>
+      </collision>
+    </link> -->
+    <!--
     <joint name="${prefix}camera_left_ir_joint" type="fixed">
       <origin
@@ -322,5 +326,5 @@
           <color rgba="0.792156862745098 0.819607843137255 0.933333333333333 1" />
         </material>
-      </visual>
+      </visual> -->
       <!-- <collision>
         <origin
@@ -330,5 +334,5 @@
           <mesh filename="${mesh_path}camera_infra2_optical_frame.STL" />
         </geometry>
-      </collision> -->
+      </collision>
     </link>
     <joint name="${prefix}camera_left_ir_optical_joint" type="fixed">
@@ -339,5 +343,5 @@
       <child link="${prefix}camera_left_ir_optical_frame" />
       <axis xyz="0 0 0" />
-    </joint>
+    </joint> -->
     <link name="${prefix}camera_depth_frame">
       <inertial>

File: src/xarm_ros2/xarm_description/urdf/dual_xarm_device.urdf.xacro (robot description, xacro)
@@ -108,5 +108,5 @@
     model1300="$(arg model1300_2)" robot_sn="$(arg robot_sn_2)" mesh_suffix="$(arg mesh_suffix)" kinematics_suffix="$(arg kinematics_suffix_2)" gripper_version="$(arg gripper_version_2)" />
   <xacro:gemini_2 prefix="$(arg prefix_2)" parent="$(arg prefix_2)link_eef"/>
-   <xacro:femto_bolt prefix="G" parent="world">
+   <xacro:femto_bolt prefix="G_camera" parent="world">
     <origin xyz="0.526 0.290 0.905" rpy="0.0 -1.3090 0.0"/>
   </xacro:femto_bolt>

File: src/xarm_ros2/xarm_moveit_config/srdf/_xarm7_macro.srdf.xacro (robot description, xacro)
@@ -57,4 +57,13 @@
       <joint name="${prefix}joint6" value="-1.3962" />
       <joint name="${prefix}joint7" value="0" />
+    </group_state>
+    <group_state name="ready_forward" group="${prefix}xarm7">
+      <joint name="${prefix}joint1" value="-0" />
+      <joint name="${prefix}joint2" value="-0.3490" />
+      <joint name="${prefix}joint3" value="-0" />
+      <joint name="${prefix}joint4" value="0.9250" />
+      <joint name="${prefix}joint5" value="0.0" />
+      <joint name="${prefix}joint6" value="0.0" />
+      <joint name="${prefix}joint7" value="0.0" />
     </group_state>
     <!-- gripper -->
