Commit message: updated file paths to be universal

File: src/xarm_ros2/orbbec_description/urdf/femto_bolt.urdf.xacro (robot description, xacro)
@@ -37,5 +37,5 @@
           <origin xyz="0 0 0" rpy="0 0 0"/>
           <geometry>
-            <mesh filename="file:///home/cadennurse/xarm_ws/src/xarm_ros2/orbbec_description/meshes/femto_bolt/femto_bolt.stl" />
+            <mesh filename="package://orbbec_description/meshes/femto_bolt/femto_bolt.stl" />
           </geometry>
           <material name="">
@@ -46,5 +46,5 @@
           <origin xyz="0 0 0" rpy="0 0 0"/>
           <geometry>
-            <mesh filename="file:///home/cadennurse/xarm_ws/src/xarm_ros2/orbbec_description/meshes/femto_bolt/femto_bolt.stl" />
+            <mesh filename="package://xarm_ws/src/xarm_ros2/orbbec_description/meshes/femto_bolt/femto_bolt.stl" />
           </geometry>
         </collision>

File: src/xarm_ros2/orbbec_description/urdf/gemini_2.urdf.xacro (robot description, xacro)
@@ -5,5 +5,5 @@
 <robot xmlns:xacro="http://ros.org/wiki/xacro" name="gemini_2">
   <xacro:macro name="gemini_2" params="prefix parent">
-    <xacro:property name="mesh_path" value="file:///home/cadennurse/xarm_ws/src/xarm_ros2/orbbec_description/meshes/gemini2/" />
+    <xacro:property name="mesh_path" value="package://orbbec_description/meshes/gemini2/" />
     <joint name="${prefix}camera_mount_joint" type="fixed">
       <origin xyz="0.06746 -0.0245 0.0237" rpy="3.1415926535897931 -1.5707963267948966 0" />
