Commit message: moveit working as the demo launch file had commented out robot state publisher. cameras need some fixing

File: src/xarm_ros2/orbbec_description/urdf/gemini_2.urdf.xacro (robot description, xacro)
@@ -37,5 +37,5 @@
         </material>
       </visual>
-      <collision>
+      <!--<collision>
         <origin
           xyz="-0.01491 -0.025 -0.0125"
@@ -44,5 +44,5 @@
           <mesh filename="${mesh_path}base_link.STL" />
         </geometry>
-      </collision>
+      </collision> -->
     </link>
     <link name="${prefix}camera_botter_screw_frame">
@@ -71,5 +71,5 @@
         </material>
       </visual>
-      <collision>
+      <!-- <collision>
         <origin
           xyz="0 0 0"
@@ -78,5 +78,5 @@
           <mesh filename="${mesh_path}camera_botter_screw_frame.STL" />
         </geometry>
-      </collision>
+      </collision> -->
     </link>
     <joint name="${prefix}camera_botter_screw_joint" type="fixed">
@@ -113,5 +113,5 @@
         </material>
       </visual>
-      <collision>
+      <!-- <collision>
         <origin
           xyz="0 0 0"
@@ -120,5 +120,5 @@
           <mesh filename="${mesh_path}camera_infra1_frame.STL" />
         </geometry>
-      </collision>
+      </collision> -->
     </link>
     <joint name="${prefix}camera_right_ir_joint" type="fixed">
@@ -155,5 +155,5 @@
         </material>
       </visual>
-      <collision>
+      <!-- <collision>
         <origin
           xyz="0 0 0"
@@ -162,5 +162,5 @@
           <mesh filename="${mesh_path}camera_infra1_optical_frame.STL" />
         </geometry>
-      </collision>
+      </collision> -->
     </link>
     <joint name="${prefix}camera_right_ir_optical_joint" type="fixed">
@@ -197,5 +197,5 @@
         </material>
       </visual>
-      <collision>
+      <!-- <collision>
         <origin
           xyz="0 0 0"
@@ -204,5 +204,5 @@
           <mesh filename="${mesh_path}camera_color_frame.STL" />
         </geometry>
-      </collision>
+      </collision> -->
     </link>
     <joint name="${prefix}camera_color_joint" type="fixed">
@@ -239,5 +239,5 @@
         </material>
       </visual>
-      <collision>
+      <!-- <collision>
         <origin
           xyz="0 0 0"
@@ -246,5 +246,5 @@
           <mesh filename="${mesh_path}camera_color_optical_frame.STL" />
         </geometry>
-      </collision>
+      </collision> -->
     </link>
     <joint name="${prefix}camera_color_optical_joint" type="fixed">
@@ -281,5 +281,5 @@
         </material>
       </visual>
-      <collision>
+      <!-- <collision>
         <origin
           xyz="0 0 0"
@@ -288,5 +288,5 @@
           <mesh filename="${mesh_path}camera_infra2_frame.STL" />
         </geometry>
-      </collision>
+      </collision> -->
     </link>
     <joint name="${prefix}camera_left_ir_joint" type="fixed">
@@ -323,5 +323,5 @@
         </material>
       </visual>
-      <collision>
+      <!-- <collision>
         <origin
           xyz="0 0 0"
@@ -330,5 +330,5 @@
           <mesh filename="${mesh_path}camera_infra2_optical_frame.STL" />
         </geometry>
-      </collision>
+      </collision> -->
     </link>
     <joint name="${prefix}camera_left_ir_optical_joint" type="fixed">
@@ -365,5 +365,5 @@
         </material>
       </visual>
-      <collision>
+      <!-- <collision>
         <origin
           xyz="0 0 0"
@@ -372,5 +372,5 @@
           <mesh filename="${mesh_path}camera_depth_frame.STL" />
         </geometry>
-      </collision>
+      </collision> -->
     </link>
     <joint name="${prefix}camera_depth_joint" type="fixed">

File: src/xarm_ros2/xarm_description/urdf/dual_xarm_device.urdf.xacro (robot description, xacro)
@@ -29,6 +29,6 @@
   <xacro:arg name="add_realsense_d435i_1" default="false"/>
   <xacro:arg name="add_realsense_d435i_2" default="false"/>
-  <xacro:arg name="add_d435i_links_1" default="true"/>
-  <xacro:arg name="add_d435i_links_2" default="true"/>
+  <xacro:arg name="add_d435i_links_1" default="false"/>
+  <xacro:arg name="add_d435i_links_2" default="false"/>
   <xacro:arg name="add_other_geometry_1" default="false"/>
   <xacro:arg name="geometry_type_1" default="box"/>
@@ -66,5 +66,6 @@
   <!-- load xarm device -->
   <xacro:include filename="$(find xarm_description)/urdf/xarm_device_macro.xacro" />
-  <xacro:include filename="$(find orbbec_description)/urdf/gemini_2.urdf.xacro" />
+  <!--<xacro:include filename="$(find orbbec_description)/urdf/gemini_2.urdf.xacro" />
+  <xacro:include filename="$(find orbbec_description)/urdf/femto_bolt.urdf.xacro" /> -->
   <xacro:xarm_device prefix="$(arg prefix_1)" hw_ns="$(arg hw_ns)" limited="$(arg limited)"
     effort_control="$(arg effort_control)" velocity_control="$(arg velocity_control)"
@@ -86,5 +87,5 @@
     baud_checkset="$(arg baud_checkset_1)" default_gripper_baud="$(arg default_gripper_baud_1)"
     model1300="$(arg model1300_1)" robot_sn="$(arg robot_sn_1)" mesh_suffix="$(arg mesh_suffix)" kinematics_suffix="$(arg kinematics_suffix_1)" gripper_version="$(arg gripper_version_1)" />
-  <xacro:gemini_2 prefix="$(arg prefix_1)" parent="$(arg prefix_1)link_eef"/>
+  <!-- <xacro:gemini_2 prefix="$(arg prefix_1)" parent="$(arg prefix_1)link_eef"/> -->
   <xacro:xarm_device prefix="$(arg prefix_2)" hw_ns="$(arg hw_ns)" limited="$(arg limited)"
     effort_control="$(arg effort_control)" velocity_control="$(arg velocity_control)"
@@ -106,4 +107,7 @@
     baud_checkset="$(arg baud_checkset_2)" default_gripper_baud="$(arg default_gripper_baud_2)"
     model1300="$(arg model1300_2)" robot_sn="$(arg robot_sn_2)" mesh_suffix="$(arg mesh_suffix)" kinematics_suffix="$(arg kinematics_suffix_2)" gripper_version="$(arg gripper_version_2)" />
-  <xacro:gemini_2 prefix="$(arg prefix_2)" parent="$(arg prefix_2)link_eef"/>
+  <!-- <xacro:gemini_2 prefix="$(arg prefix_2)" parent="$(arg prefix_2)link_eef"/> -->
+  <!-- <xacro:femto_bolt prefix="G" parent="world">
+    <origin xyz="0.526 0.290 0.905" rpy="0.0 -1.3090 1.5708"/>
+  </xacro:femto_bolt> -->
 </robot>

Commit message: added gripper controllers, removed bio, vacuum, and robotiq grippers

File: src/xarm_ros2/orbbec_description/urdf/gemini_2.urdf.xacro (robot description, xacro)
@@ -7,5 +7,5 @@
     <xacro:property name="mesh_path" value="file:///home/cadennurse/xarm_ws/src/xarm_ros2/orbbec_description/meshes/gemini2/" />
     <joint name="${prefix}camera_mount_joint" type="fixed">
-      <origin xyz="0.06746 -0.0175 0.0237" rpy="3.1415926535897931 -1.5707963267948966 0" />
+      <origin xyz="0.06746 -0.0245 0.0237" rpy="3.1415926535897931 -1.5707963267948966 0" />
       <parent link="${parent}" />
       <child link="${prefix}camera_link" />
