Commit message: addtional apriltag setup for manipulation of a basic object. transforms are functional with a world pose set to L_xarm_base_link and workspace_origin set to tag_4

File: src/xarm_ros2/orbbec_description/urdf/gemini_2.urdf.xacro (robot description, xacro)
@@ -37,12 +37,13 @@
         </material>
       </visual>
-      <!--<collision>
+      <collision>
         <origin
           xyz="-0.01491 -0.025 -0.0125"
           rpy="0 0 0" />
         <geometry>
-          <mesh filename="${mesh_path}base_link.STL" />
-        </geometry>
-      </collision> -->
+          <!-- <mesh filename="${mesh_path}base_link.STL" /> -->
+          <box size="0.001 0.001 0.001" />
+        </geometry>
+      </collision>
     </link>
     <link name="${prefix}camera_botter_screw_frame">
@@ -71,12 +72,13 @@
         </material>
       </visual>
-      <!-- <collision>
-        <origin
-          xyz="0 0 0"
-          rpy="0 0 0" />
-        <geometry>
-          <mesh filename="${mesh_path}camera_botter_screw_frame.STL" />
-        </geometry>
-      </collision> -->
+      <collision>
+        <origin
+          xyz="0.002 0 0"
+          rpy="0 0 0" />
+        <geometry>
+          <!-- <mesh filename="${mesh_path}camera_botter_screw_frame.STL" /> -->
+          <box size="0.001 0.001 0.001" />
+        </geometry>
+      </collision>
     </link>
     <joint name="${prefix}camera_botter_screw_joint" type="fixed">
@@ -199,12 +201,13 @@
         </material>
       </visual>
-      <!-- <collision>
-        <origin
-          xyz="0 0 0"
-          rpy="0 0 0" />
-        <geometry>
-          <mesh filename="${mesh_path}camera_color_frame.STL" />
-        </geometry>
-      </collision> -->
+      <collision>
+        <origin
+          xyz="0.04 0 0"
+          rpy="0 0 0" />
+        <geometry>
+          <!-- <mesh filename="${mesh_path}camera_color_frame.STL" /> -->
+          <box size="0.001 0.001 0.001" />
+        </geometry>
+      </collision>
     </link>
     <joint name="${prefix}camera_color_joint" type="fixed">
@@ -241,12 +244,13 @@
         </material>
       </visual>
-      <!-- <collision>
-        <origin
-          xyz="0 0 0"
-          rpy="0 0 0" />
-        <geometry>
-          <mesh filename="${mesh_path}camera_color_optical_frame.STL" />
-        </geometry>
-      </collision> -->
+      <collision>
+        <origin
+          xyz="0 0.02 0"
+          rpy="0 0 0" />
+        <geometry>
+          <!-- <mesh filename="${mesh_path}camera_color_optical_frame.STL" /> -->
+          <box size="0.001 0.001 0.001" />
+        </geometry>
+      </collision>
     </link>
     <joint name="${prefix}camera_color_optical_joint" type="fixed">
@@ -369,12 +373,13 @@
         </material>
       </visual>
-      <!-- <collision>
-        <origin
-          xyz="0 0 0"
-          rpy="0 0 0" />
-        <geometry>
-          <mesh filename="${mesh_path}camera_depth_frame.STL" />
-        </geometry>
-      </collision> -->
+      <collision>
+        <origin
+          xyz="0 0.04 0"
+          rpy="0 0 0" />
+        <geometry>
+          <!-- <mesh filename="${mesh_path}camera_depth_frame.STL" /> -->
+          <box size="0.001 0.001 0.001" />
+        </geometry>
+      </collision>
     </link>
     <joint name="${prefix}camera_depth_joint" type="fixed">
