Commit message: added a wall in rviz

File: src/xarm_ros2/xarm_description/urdf/gripper/xarm_gripper.urdf.xacro (robot description, xacro)
@@ -56,5 +56,5 @@
       <child link="${prefix}left_outer_knuckle" />
       <axis xyz="1 0 0" />
-      <limit lower="0" upper="0.85" effort="50" velocity="2" />
+      <limit lower="0" upper="0.855" effort="50" velocity="2" />
     </joint>
     <link name="${prefix}left_finger">
@@ -81,5 +81,5 @@
       <child link="${prefix}left_finger" />
       <axis xyz="-1 0 0" />
-      <limit lower="0" upper="0.85" effort="50" velocity="2" />
+      <limit lower="0" upper="0.855" effort="50" velocity="2" />
       <mimic joint="${prefix}drive_joint" multiplier="1" offset="0" />
     </joint>
@@ -107,5 +107,5 @@
       <child link="${prefix}left_inner_knuckle" />
       <axis xyz="1 0 0" />
-      <limit lower="0" upper="0.85" effort="50" velocity="2" />
+      <limit lower="0" upper="0.855" effort="50" velocity="2" />
       <mimic joint="${prefix}drive_joint" multiplier="1" offset="0" />
     </joint>
@@ -133,5 +133,5 @@
       <child link="${prefix}right_outer_knuckle" />
       <axis xyz="-1 0 0" />
-      <limit lower="0" upper="0.85" effort="50" velocity="2" />
+      <limit lower="0" upper="0.855" effort="50" velocity="2" />
       <mimic joint="${prefix}drive_joint" multiplier="1" offset="0" />
     </joint>
@@ -159,5 +159,5 @@
       <child link="${prefix}right_finger" />
       <axis xyz="1 0 0" />
-      <limit lower="0" upper="0.85" effort="50" velocity="2" />
+      <limit lower="0" upper="0.855" effort="50" velocity="2" />
       <mimic joint="${prefix}drive_joint" multiplier="1" offset="0" />
     </joint>
@@ -185,5 +185,5 @@
       <child link="${prefix}right_inner_knuckle" />
       <axis xyz="-1 0 0" />
-      <limit lower="0" upper="0.85" effort="50" velocity="2" />
+      <limit lower="0" upper="0.855" effort="50" velocity="2" />
       <mimic joint="${prefix}drive_joint" multiplier="1" offset="0" />
     </joint>
