Commit message: rviz now runs with all cameras with rgb and pointcloud. no issues but fps slow

File: src/xarm_ros2/xarm_description/urdf/dual_xarm_device.urdf.xacro (robot description, xacro)
@@ -109,5 +109,5 @@
   <xacro:gemini_2 prefix="$(arg prefix_2)" parent="$(arg prefix_2)link_eef"/>
    <xacro:femto_bolt prefix="G_camera" parent="world">
-    <origin xyz="0.526 0.290 0.905" rpy="0.0 -1.3090 0.0"/>
+    <origin xyz="0.526 0.290 0.905" rpy="0.0 1.3090 3.1416"/>
   </xacro:femto_bolt>
 </robot>

Commit message: moved global camera to ailgn with physical arms better using depth cloud

File: src/xarm_ros2/xarm_description/urdf/dual_xarm_device.urdf.xacro (robot description, xacro)
@@ -94,5 +94,5 @@
     ros2_control_plugin="$(arg ros2_control_plugin)" robot_type="$(arg robot_type_2)"
     load_gazebo_plugin="true" ros2_control_params="$(arg ros2_control_params)"
-    attach_to="world" attach_xyz="0 0.548 0" attach_rpy="0 0 0" create_attach_link="false"
+    attach_to="world" attach_xyz="0 0.55 0" attach_rpy="0 0 0" create_attach_link="false"
     add_realsense_d435i="$(arg add_realsense_d435i_2)"
     add_d435i_links="$(arg add_d435i_links_2)"
@@ -109,5 +109,5 @@
   <xacro:gemini_2 prefix="$(arg prefix_2)" parent="$(arg prefix_2)link_eef"/>
    <xacro:femto_bolt prefix="G_camera" parent="world">
-    <origin xyz="0.526 0.290 0.905" rpy="0.0 1.3090 3.1416"/>
+    <origin xyz="0.526 0.290 0.885" rpy="0.0 1.3090 3.1416"/>
   </xacro:femto_bolt>
 </robot>

Commit message: more accurate global camera postion

File: src/xarm_ros2/xarm_description/urdf/dual_xarm_device.urdf.xacro (robot description, xacro)
@@ -109,5 +109,5 @@
   <xacro:gemini_2 prefix="$(arg prefix_2)" parent="$(arg prefix_2)link_eef"/>
    <xacro:femto_bolt prefix="G_camera" parent="world">
-    <origin xyz="0.526 0.290 0.885" rpy="0.0 1.3090 3.1416"/>
+    <origin xyz="0.526 0.280 0.885" rpy="0.0 1.3090 3.1416"/>
   </xacro:femto_bolt>
 </robot>

Commit message: small changes to improve efficiency with topics

File: src/xarm_ros2/xarm_description/urdf/dual_xarm_device.urdf.xacro (robot description, xacro)
@@ -109,5 +109,5 @@
   <xacro:gemini_2 prefix="$(arg prefix_2)" parent="$(arg prefix_2)link_eef"/>
    <xacro:femto_bolt prefix="G_camera" parent="world">
-    <origin xyz="0.526 0.280 0.885" rpy="0.0 1.3090 3.1416"/>
+    <origin xyz="0.535 0.270 0.875" rpy="0.0 1.3090 3.1416"/>
   </xacro:femto_bolt>
 </robot>
