Commit message: task planning working. added xarm-python-sdk for hardware debugging. be cautious of Safety Boundaries

File: src/xarm_ros2/xarm_description/urdf/dual_xarm_device.urdf.xacro (robot description, xacro)
@@ -74,5 +74,5 @@
     ros2_control_plugin="$(arg ros2_control_plugin)" robot_type="$(arg robot_type_1)"
     load_gazebo_plugin="false" ros2_control_params="$(arg ros2_control_params)"
-    attach_to="world" attach_xyz="0 0 0" attach_rpy="0 0 0"
+    attach_to="world" attach_xyz="0 0 0.01" attach_rpy="0 0 0"
     add_realsense_d435i="$(arg add_realsense_d435i_1)"
     add_d435i_links="$(arg add_d435i_links_1)"
@@ -94,5 +94,5 @@
     ros2_control_plugin="$(arg ros2_control_plugin)" robot_type="$(arg robot_type_2)"
     load_gazebo_plugin="true" ros2_control_params="$(arg ros2_control_params)"
-    attach_to="world" attach_xyz="0 0.55 0" attach_rpy="0 0 0" create_attach_link="false"
+    attach_to="world" attach_xyz="0 0.546 0.01" attach_rpy="0 0 0" create_attach_link="false"
     add_realsense_d435i="$(arg add_realsense_d435i_2)"
     add_d435i_links="$(arg add_d435i_links_2)"
@@ -109,5 +109,5 @@
   <xacro:gemini_2 prefix="$(arg prefix_2)" parent="$(arg prefix_2)link_eef"/>
    <xacro:femto_bolt prefix="G_camera" parent="world">
-    <origin xyz="0.535 0.270 0.875" rpy="0.0 1.3090 3.1416"/>
+    <origin xyz="0.535 0.270 0.884" rpy="0.0 1.308996939 3.1416"/>
   </xacro:femto_bolt>
 </robot>

File: src/xarm_ros2/xarm_moveit_config/srdf/_xarm7_macro.srdf.xacro (robot description, xacro)
@@ -68,20 +68,20 @@
     </group_state>
     <group_state name="prepare_L" group="${prefix}xarm7">
-      <joint name="${prefix}joint1" value="-1.0472" />
-      <joint name="${prefix}joint2" value="0.8378" />
-      <joint name="${prefix}joint3" value="0.4712" />
-      <joint name="${prefix}joint4" value="1.5359" />
-      <joint name="${prefix}joint5" value="-2.4435" />
-      <joint name="${prefix}joint6" value="-1.6920" />
-      <joint name="${prefix}joint7" value="0.7330" />
+      <joint name="${prefix}joint1" value="-1.8675" />
+      <joint name="${prefix}joint2" value="0.9250" />
+      <joint name="${prefix}joint3" value="1.4137" />
+      <joint name="${prefix}joint4" value="1.2915" />
+      <joint name="${prefix}joint5" value="0.4189" />
+      <joint name="${prefix}joint6" value="1.6755" />
+      <joint name="${prefix}joint7" value="4.3982" />
     </group_state>
     <group_state name="prepare_R" group="${prefix}xarm7">
-      <joint name="${prefix}joint1" value="1.1345" />
-      <joint name="${prefix}joint2" value="1.0821" />
-      <joint name="${prefix}joint3" value="-0.7330" />
-      <joint name="${prefix}joint4" value="1.9199" />
-      <joint name="${prefix}joint5" value="2.7402" />
-      <joint name="${prefix}joint6" value="-1.6920" />
-      <joint name="${prefix}joint7" value="-1.0472" />
+      <joint name="${prefix}joint1" value="-1.4835" />
+      <joint name="${prefix}joint2" value="-0.7505" />
+      <joint name="${prefix}joint3" value="2.1118" />
+      <joint name="${prefix}joint4" value="1.3265" />
+      <joint name="${prefix}joint5" value="-0.3840" />
+      <joint name="${prefix}joint6" value="1-6581" />
+      <joint name="${prefix}joint7" value="2.1468" />
     </group_state>
     <!-- gripper -->

Commit message: laptop manipulation progress. urdf visable and mtc node generated. working on geometry correction.

File: src/xarm_ros2/xarm_description/urdf/dual_xarm_device.urdf.xacro (robot description, xacro)
@@ -68,4 +68,5 @@
   <xacro:include filename="$(find orbbec_description)/urdf/gemini_2.urdf.xacro" /> <!-- _collision.urdf for collision geometry of the gemini 2 -->
   <xacro:include filename="$(find orbbec_description)/urdf/femto_bolt.urdf.xacro" />
+  <!-- <xacro:include filename="$(find xarm_description)/other/thinkpad_x13_gen1.urdf.xacro" />  STUPID LAPTOP Hardcode -->
   <xacro:xarm_device prefix="$(arg prefix_1)" hw_ns="$(arg hw_ns)" limited="$(arg limited)"
     effort_control="$(arg effort_control)" velocity_control="$(arg velocity_control)"
@@ -111,3 +112,7 @@
     <origin xyz="0.535 0.270 0.884" rpy="0.0 1.308996939 3.1416"/>
   </xacro:femto_bolt>
+<!--
+  <xacro:laptop parent="world">
+    <origin xyz="0 0 0" rpy="0 0 0"/>
+  </xacro:laptop> -->
 </robot>

File: src/xarm_ros2/xarm_moveit_config/dual_config/config/_xarm7_macro.srdf.xacro (robot description, xacro)
@@ -102,4 +102,13 @@
       <joint name="${prefix}joint6" value="-1.55" />
       <joint name="${prefix}joint7" value="1.95" />
+    </group_state>
+    <group_state name="pre_handover_R" group="R_xarm7">
+      <joint name="R_joint1" value="-1.0821" />
+      <joint name="R_joint2" value="-1.0821" />
+      <joint name="R_joint3" value="1.2217" />
+      <joint name="R_joint4" value="0.6981" />
+      <joint name="R_joint5" value="-0.6283" />
+      <joint name="R_joint6" value="1.1345" />
+      <joint name="R_joint7" value="1.6930" />
     </group_state>
     <!-- gripper -->
