Commit message: pick and place with apriltag box works. good efficency and progress

File: src/xarm_ros2/xarm_moveit_config/dual_config/config/_xarm7_macro.srdf.xacro (robot description, xacro)
@@ -73,5 +73,5 @@
       <joint name="${prefix}joint4" value="1.2915" />
       <joint name="${prefix}joint5" value="0.4189" />
-      <joint name="${prefix}joint6" value="1.6755" />
+      <joint name="${prefix}joint6" value="-1.6755" />
       <joint name="${prefix}joint7" value="4.3982" />
     </group_state>
@@ -82,5 +82,5 @@
       <joint name="${prefix}joint4" value="1.3265" />
       <joint name="${prefix}joint5" value="-0.3840" />
-      <joint name="${prefix}joint6" value="1-6581" />
+      <joint name="${prefix}joint6" value="-1.6581" />
       <joint name="${prefix}joint7" value="2.1468" />
     </group_state>

File: src/xarm_ros2/xarm_moveit_config/srdf/_xarm7_macro.srdf.xacro (robot description, xacro)
@@ -82,5 +82,5 @@
       <joint name="${prefix}joint4" value="1.3265" />
       <joint name="${prefix}joint5" value="-0.3840" />
-      <joint name="${prefix}joint6" value="1-6581" />
+      <joint name="${prefix}joint6" value="-1.6581" />
       <joint name="${prefix}joint7" value="2.1468" />
     </group_state>

Commit message: Safe handover files and updated cmake to accomidate. Shoff has issues with connect stages not getting solutions.

File: src/xarm_ros2/xarm_moveit_config/dual_config/config/_xarm7_macro.srdf.xacro (robot description, xacro)
@@ -84,4 +84,31 @@
       <joint name="${prefix}joint6" value="-1.6581" />
       <joint name="${prefix}joint7" value="2.1468" />
+    </group_state>
+    <group_state name="pre_handover_R" group="${prefix}xarm7">
+      <joint name="${prefix}joint1" value="-1.10" />
+      <joint name="${prefix}joint2" value="-0.45" />
+      <joint name="${prefix}joint3" value="1.85" />
+      <joint name="${prefix}joint4" value="1.10" />
+      <joint name="${prefix}joint5" value="-0.20" />
+      <joint name="${prefix}joint6" value="-1.45" />
+      <joint name="${prefix}joint7" value="1.85" />
+    </group_state>
+    <group_state name="post_handover_L" group="${prefix}xarm7">
+      <joint name="${prefix}joint1" value="-1.55" />
+      <joint name="${prefix}joint2" value="0.70" />
+      <joint name="${prefix}joint3" value="1.55" />
+      <joint name="${prefix}joint4" value="1.20" />
+      <joint name="${prefix}joint5" value="0.30" />
+      <joint name="${prefix}joint6" value="-1.55" />
+      <joint name="${prefix}joint7" value="3.80" />
+    </group_state>
+    <group_state name="pre_place_R" group="${prefix}xarm7">
+      <joint name="${prefix}joint1" value="-1.20" />
+      <joint name="${prefix}joint2" value="-0.95" />
+      <joint name="${prefix}joint3" value="1.95" />
+      <joint name="${prefix}joint4" value="1.30" />
+      <joint name="${prefix}joint5" value="-0.25" />
+      <joint name="${prefix}joint6" value="-1.55" />
+      <joint name="${prefix}joint7" value="1.95" />
     </group_state>
     <!-- gripper -->

Commit message: Shoff finds a solution and works.

File: src/xarm_ros2/xarm_moveit_config/dual_config/config/_xarm7_macro.srdf.xacro (robot description, xacro)
@@ -73,26 +73,17 @@
       <joint name="${prefix}joint4" value="1.2915" />
       <joint name="${prefix}joint5" value="0.4189" />
-      <joint name="${prefix}joint6" value="-1.6755" />
+      <joint name="${prefix}joint6" value="1.6755" />
       <joint name="${prefix}joint7" value="4.3982" />
     </group_state>
     <group_state name="prepare_R" group="${prefix}xarm7">
-      <joint name="${prefix}joint1" value="-1.4835" />
-      <joint name="${prefix}joint2" value="-0.7505" />
-      <joint name="${prefix}joint3" value="2.1118" />
-      <joint name="${prefix}joint4" value="1.3265" />
-      <joint name="${prefix}joint5" value="-0.3840" />
-      <joint name="${prefix}joint6" value="-1.6581" />
-      <joint name="${prefix}joint7" value="2.1468" />
-    </group_state>
-    <group_state name="pre_handover_R" group="${prefix}xarm7">
-      <joint name="${prefix}joint1" value="-1.10" />
-      <joint name="${prefix}joint2" value="-0.45" />
-      <joint name="${prefix}joint3" value="1.85" />
-      <joint name="${prefix}joint4" value="1.10" />
-      <joint name="${prefix}joint5" value="-0.20" />
-      <joint name="${prefix}joint6" value="-1.45" />
-      <joint name="${prefix}joint7" value="1.85" />
-    </group_state>
-    <group_state name="post_handover_L" group="${prefix}xarm7">
+      <joint name="${prefix}joint1" value="-1.3793" />
+      <joint name="${prefix}joint2" value="-0.6632" />
+      <joint name="${prefix}joint3" value="2.0420" />
+      <joint name="${prefix}joint4" value="1.3963" />
+      <joint name="${prefix}joint5" value="-0.5061" />
+      <joint name="${prefix}joint6" value="1.8326" />
+      <joint name="${prefix}joint7" value="2.0769" />
+    </group_state>
+    <group_state name="out_of_the_way_L" group="${prefix}xarm7">
       <joint name="${prefix}joint1" value="-1.55" />
       <joint name="${prefix}joint2" value="0.70" />
@@ -103,5 +94,5 @@
       <joint name="${prefix}joint7" value="3.80" />
     </group_state>
-    <group_state name="pre_place_R" group="${prefix}xarm7">
+    <group_state name="out_of_the_way_R" group="${prefix}xarm7">
       <joint name="${prefix}joint1" value="-1.20" />
       <joint name="${prefix}joint2" value="-0.95" />

File: src/xarm_ros2/xarm_moveit_config/srdf/_xarm7_macro.srdf.xacro (robot description, xacro)
@@ -77,11 +77,29 @@
     </group_state>
     <group_state name="prepare_R" group="${prefix}xarm7">
-      <joint name="${prefix}joint1" value="-1.4835" />
-      <joint name="${prefix}joint2" value="-0.7505" />
-      <joint name="${prefix}joint3" value="2.1118" />
-      <joint name="${prefix}joint4" value="1.3265" />
-      <joint name="${prefix}joint5" value="-0.3840" />
-      <joint name="${prefix}joint6" value="-1.6581" />
-      <joint name="${prefix}joint7" value="2.1468" />
+      <joint name="${prefix}joint1" value="-1.3793" />
+      <joint name="${prefix}joint2" value="-0.6632" />
+      <joint name="${prefix}joint3" value="2.0420" />
+      <joint name="${prefix}joint4" value="1.3963" />
+      <joint name="${prefix}joint5" value="-0.5061" />
+      <joint name="${prefix}joint6" value="1.8326" />
+      <joint name="${prefix}joint7" value="2.0769" />
+    </group_state>
+    <group_state name="out_of_the_way_L" group="${prefix}xarm7">
+      <joint name="${prefix}joint1" value="-1.55" />
+      <joint name="${prefix}joint2" value="0.70" />
+      <joint name="${prefix}joint3" value="1.55" />
+      <joint name="${prefix}joint4" value="1.20" />
+      <joint name="${prefix}joint5" value="0.30" />
+      <joint name="${prefix}joint6" value="-1.55" />
+      <joint name="${prefix}joint7" value="3.80" />
+    </group_state>
+    <group_state name="out_of_the_way_R" group="${prefix}xarm7">
+      <joint name="${prefix}joint1" value="-1.20" />
+      <joint name="${prefix}joint2" value="-0.95" />
+      <joint name="${prefix}joint3" value="1.95" />
+      <joint name="${prefix}joint4" value="1.30" />
+      <joint name="${prefix}joint5" value="-0.25" />
+      <joint name="${prefix}joint6" value="-1.55" />
+      <joint name="${prefix}joint7" value="1.95" />
     </group_state>
     <!-- gripper -->
