Commit message: Rviz now can visualize laptop being opened past 90 degrees. cannot function when less than 90

File: src/xarm_ros2/xarm_description/urdf/other/thinkpad_x13_gen1.urdf.xacro (robot description, xacro)
@@ -52,5 +52,5 @@
   <link name="lid_link">
     <inertial>
-      <origin xyz="0 ${lid_length / 2.0} ${lid_thickness / 2.0}" rpy="0 0 0"/>
+      <origin xyz="0 ${lid_width / 2.0} ${lid_thickness / 2.0}" rpy="0 0 0"/>
       <mass value="${lid_mass}"/>
       <inertia
@@ -63,5 +63,5 @@
     </inertial>
     <visual>
-      <origin xyz="0 ${lid_length / 2.0} ${lid_thickness / 2.0}" rpy="0 0 0"/>
+      <origin xyz="0 ${lid_width/ 2.0} ${lid_thickness / 2.0}" rpy="0 0 0"/>
       <geometry>
         <box size="${lid_length} ${lid_width} ${lid_thickness}"/>
@@ -70,5 +70,5 @@
     </visual>
     <collision>
-      <origin xyz="0 ${lid_length / 2.0} ${lid_thickness / 2.0}" rpy="0 0 0"/>
+      <origin xyz="0 ${lid_width / 2.0} ${lid_thickness / 2.0}" rpy="0 0 0"/>
       <geometry>
         <box size="${lid_length} ${lid_width} ${lid_thickness}"/>

Commit message: already working 10 times better. matching tag names and proper angles

File: src/xarm_ros2/xarm_description/urdf/other/thinkpad_x13_gen1.urdf.xacro (robot description, xacro)
@@ -11,5 +11,5 @@
   <xacro:property name="hinge_x" value="0.0"/>
   <xacro:property name="hinge_y" value="-0.1085"/>
-  <xacro:property name="hinge_z" value="0.015"/>
+  <xacro:property name="hinge_z" value="${base_thickness}"/>
   <material name="base_red">
     <color rgba="1 0 0 1"/>
@@ -18,5 +18,7 @@
     <color rgba="0 0 1 1"/>
   </material>
+  <!-- Dummy link for inertia -->
   <link name="laptop_world"/>
+  <!-- Base -->
   <link name="laptop_base_link">
     <inertial>
@@ -45,4 +47,5 @@
     </collision>
   </link>
+  <!-- Dummy joint to link inertia -->
   <joint name="laptop_world_to_base" type="fixed">
     <parent link="laptop_world"/>
@@ -50,4 +53,5 @@
     <origin xyz="0 0 0" rpy="0 0 0"/>
   </joint>
+  <!-- Lid/Screen -->
   <link name="lid_link">
     <inertial>
@@ -76,4 +80,5 @@
     </collision>
   </link>
+  <!-- Hinge Joint -->
   <joint name="hinge_joint" type="revolute">
     <parent link="laptop_base_link"/>
@@ -83,3 +88,32 @@
     <limit lower="0.0" upper="3.1416" effort="1.0" velocity="1.0"/>
   </joint>
+    <!-- Reference frames -->
+  <!-- <link name="hinge"/>
+  <joint name="base_to_hinge" type="fixed">
+    <parent link="base_link"/>
+    <child link="hinge"/>
+    <origin xyz="${hinge_x} ${hinge_y} ${hinge_z}" rpy="0 0 0"/>
+  </joint> -->
+    <!-- Base tag centered on top plane of base -->
+     <!-- might need [1.5708, 3.1416, 1.5708] -->
+  <link name="tag_laptop_base"/>
+  <joint name="base_to_base_tag" type="fixed">
+    <parent link="laptop_base_link"/>
+    <child link="tag_laptop_base"/>
+    <origin xyz="0 0 ${base_thickness}" rpy="0 0 0"/>
+  </joint>
+  <!-- Lid outer tag centered on outside plane -->
+  <link name="tag_laptop_lid_inner"/>
+  <joint name="lid_to_inner_tag" type="fixed">
+    <parent link="lid_link"/>
+    <child link="tag_laptop_lid_inner"/>
+    <origin xyz="${lid_length} ${lid_width / 2.0} -${lid_thickness}" rpy="0 0 0"/>
+  </joint>
+  <!-- Lid inner tag centered on inside plane -->
+  <link name="tag_laptop_lid_outer"/>
+  <joint name="lid_to_outer_tag" type="fixed">
+    <parent link="lid_link"/>
+    <child link="tag_laptop_lid_outer"/>
+    <origin xyz="${lid_length} ${lid_width / 2.0} ${lid_thickness}" rpy="3.14159265359 3.14159265359 0"/>
+  </joint>
 </robot>
